File: boss_DS1.kicad_pcb (KiCad board)
At the start: 2 copper layers, 80 x 100 mm, 85 parts, among them J1 NMJ6HHD2, J2 NMJ6HHD2, J3 Conn_01x05, J4 Conn_01x05, J5 Conn_01x05, J6 Barrel_Jack_MountingPin, P1 boss_DS1_front_panel, Q1 MMBT5551, Q2 MMBT5551, Q3 MMBT5551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

Commit message: Fix
Parts:
- SW1: value SW_DPDT_x2 -> pedala_switch; footprint switch:switch_DPDT -> pedale:switch_DPDT
- moved SW1 0.10 mm to (85.0, 122.4)

Commit message: oK
Parts:
- removed R26: 10k, Resistor_SMD:R_0603_1608Metric_Pad0.98x0.95mm_HandSolder
Connections:
- C22 pad 2: Net-(Q4-C) -> BJT_GAIN
- D6 pad 2: 0 -> 4V5
- D7 pad 1: 0 -> 4V5
- Q4 pad 3: Net-(Q4-C) -> BJT_GAIN
- R12 pad 2: Net-(Q4-C) -> BJT_GAIN
- R25 pad 2: Net-(Q4-C) -> BJT_GAIN

Commit message: rutiranje v1.
Parts:
- moved R13 34.1 mm to (63.7, 69.1), turned to 0 degrees
- moved R18 34.1 mm to (99.5, 55.9), turned to 90 degrees
- moved R15 29.5 mm to (67.5, 65.6)
- moved D4 28.5 mm to (98.0, 78.4), turned to 180 degrees
- moved Q1 25.8 mm to (67.6, 68.4)
- moved C9 25.1 mm to (63.6, 67.4)
- moved R17 23.2 mm to (67.0, 72.1), turned to -90 degrees
- moved D7 19.5 mm to (107.5, 73.0), turned to 90 degrees
- moved R10 17.8 mm to (98.5, 60.5), turned to 90 degrees
- moved R6 17.7 mm to (108.0, 62.0), turned to 90 degrees
- moved C20 17.3 mm to (107.2, 59.2)
- moved C22 17.2 mm to (102.3, 65.7), turned to -90 degrees
- moved D6 16.6 mm to (109.8, 72.8), turned to -90 degrees
- moved U1 15.6 mm to (104.2, 77.8)
- moved R4 15.2 mm to (111.3, 59.0)
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Routing:
- net Net-(J5-Pin_4): track 0.00 -> 86.6 mm, vias 0 -> 4
- net Net-(SW1A-C): track 0.00 -> 80.9 mm
- net Net-(J1-PadT): track 0.00 -> 69.7 mm
- net Net-(C11-Pad2): track 0.00 -> 65.5 mm
- net /SW_ON: track 0.00 -> 63.7 mm, vias 0 -> 1
- net OP_OUT: track 0.00 -> 54.5 mm, vias 0 -> 4
- net /SW_MID: track 0.00 -> 53.2 mm, vias 0 -> 2
- net IN_BUFF: track 0.00 -> 29.2 mm
- net Net-(J3-Pin_1): track 0.00 -> 28.1 mm
- net Net-(U1B--): track 0.00 -> 25.7 mm
- net BJT_GAIN: track 0.00 -> 15.7 mm
- net Net-(Q3-B): track 0.00 -> 14.6 mm
- net Net-(Q4-B): track 0.00 -> 13.4 mm
- net Net-(D3-A): track 0.00 -> 12.4 mm
- net Net-(BT1-+): track 0.00 -> 10.2 mm
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
Commit message: rutiranje v2.
Parts:
- moved C7 8.23 mm to (107.3, 68.5)
- moved D7 8.23 mm to (104.0, 65.5)
- moved R14 8.23 mm to (108.4, 65.5)
- moved C21 8.23 mm to (105.5, 62.6)
- moved D6 8.23 mm to (106.2, 65.4)
- moved C27 6.89 mm to (92.2, 73.4)
- moved R10 5.73 mm to (96.2, 65.8), turned to -90 degrees
- moved R25 4.08 mm to (101.7, 69.0)
- moved R3 3.98 mm to (97.7, 76.2), turned to 90 degrees
- moved C22 3.50 mm to (98.9, 64.8), turned to 0 degrees
- moved R12 3.34 mm to (98.9, 66.4)
- moved C19 3.34 mm to (94.9, 69.0)
- moved R24 3.34 mm to (98.7, 72.7)
- moved R27 3.34 mm to (95.9, 72.0)
- moved C23 3.34 mm to (93.1, 70.8)
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Routing:
- net TONE_OUT: track 0.00 -> 26.4 mm
- net Net-(U1B--): track 25.7 -> 20.2 mm
- net Net-(Q4-B): track 13.4 -> 8.55 mm
- net Net-(J3-Pin_1): track 28.1 -> 31.9 mm, vias 0 -> 2
- net Net-(SW1A-C): track 80.9 -> 77.1 mm
- net BJT_GAIN: track 15.7 -> 12.8 mm
- net OP_OUT: track 54.5 -> 52.1 mm, vias 4 -> 0
- net Net-(J5-Pin_4): track 86.6 -> 87.9 mm
- net Net-(C11-Pad2): track 65.5 -> 64.4 mm
- net IN_BUFF: track 29.2 -> 30.2 mm
- net /SW_ON: vias 1 -> 4

Commit message: Rutiranje v3
Parts:
- moved C17 23.0 mm to (108.3, 74.4), turned to -90 degrees
- moved C26 3.68 mm to (61.3, 62.0), turned to -90 degrees
- moved R30 0.11 mm to (63.0, 62.0)
Routing:
- net 9V: track 0.00 -> 189.6 mm, vias 0 -> 8
- net 4V5: track 0.00 -> 110.4 mm, vias 0 -> 8
- net 0: track 0.00 -> 23.0 mm, vias 0 -> 18
- net Net-(J5-Pin_4): track 87.9 -> 75.2 mm
- net OP_OUT: track 52.1 -> 54.5 mm
- net Net-(J4-Pin_1): track 6.31 -> 7.99 mm
- net Net-(U1B--): track 20.2 -> 21.8 mm
- net Net-(J1-PadT): track 69.7 -> 71.2 mm
- net Net-(J3-Pin_1): track 31.9 -> 32.7 mm
- net IN_BUFF: track 30.2 -> 29.5 mm
- net /SW_ON: track 63.7 -> 64.2 mm

Commit message: verzija v4
Routing:
- net 9V: track 189.6 -> 192.2 mm

Commit message: a
Routing:
- net /SW_ON: track 64.2 -> 63.7 mm
Changed lines of the file:
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@@
 	)
 	(segment
-		(start 85.5 59)
-		(end 85.5875 59)
+		(start 85 59.5875)
+		(end 85.1 59.4875)
 		(width 0.5)
 		(layer "F.Cu")
@@
 	)
 	(segment
-		(start 85.2875 59.3)
-		(end 85.8 59.3)
+		(start 85 71.4)
+		(end 85 77.25)
+		(width 0.5)
+		(layer "F.Cu")
+		(net 25)
+	)
+	(segment
+		(start 85.1 59.4)
+		(end 85.5 59)
+		(width 0.5)
+		(layer "F.Cu")
+		(net 25)
+	)
+	(segment
+		(start 85.5 59)
+		(end 85.5875 59)
 		(width 0.5)
 		(layer "F.Cu")
@@
 	)
 	(segment
-		(start 85 71.4)
-		(end 85 77.25)
+		(start 85.1 59.4875)
+		(end 85.1 59.4)
 		(width 0.5)
 		(layer "F.Cu")
-		(net 25)
-	)
-	(segment
-		(start 85.8 59.3)
-		(end 85.5 59)
-		(width 0.5)
-		(layer "F.Cu")
-		(net 25)
-	)
-	(segment
-		(start 85 59.5875)
-		(end 85.2875 59.3)
-		(width 0.5)
-		(layer "F.Cu")

Commit message: All errors fixed
Parts:
- removed J1: NMJ6HHD2, Connector_Audio:Jack_6.35mm_Neutrik_NMJ6HHD2_Horizontal
- added J7: Conn_01x01_Socket, TestPoint:TestPoint_THTPad_D2.5mm_Drill1.2mm, F.Cu at (68.6, 89.9)
- added J8: Conn_01x01_Socket, TestPoint:TestPoint_THTPad_D2.5mm_Drill1.2mm, F.Cu at (68.5, 102.4)
- added J9: Barrel_Jack_Switch, pedale:BarrelJack, F.Cu at (63.9, 103.3)
- J2: value NMJ6HHD2 -> Jack_6.35; footprint Connector_Audio:Jack_6.35mm_Neutrik_NMJ6HHD2_Horizontal -> pedale:Jack_6.35mm
- J6: value Barrel_Jack_MountingPin -> Jack_6.35; footprint Connector_BarrelJack:BarrelJack_GCT_DCJ200-10-A_Horizontal -> pedale:Jack_6.35mm
- SW1: footprint pedale:switch_DPDT -> pedale:foot_switch_tht_and_floating
- moved J6 30.0 mm to (67.2, 133.1), turned to 180 degrees
- moved SW1 5.64 mm to (90.0, 125.0)
- moved BT1 4.61 mm to (75.0, 89.7)
- moved U1 1.55 mm to (105.4, 77.4)
- moved C10 1.21 mm to (100.9, 75.9), turned to -90 degrees
- moved C17 0.94 mm to (107.5, 73.9), turned to 0 degrees
- moved D4 0.42 mm to (99.2, 79.1)
Connections:
- BT1 pad 2: 0 -> Net-(BT1--)
- R13 pad 2: Net-(J1-PadT) -> Net-(J6-PadT)
Routing:
- net Net-(J6-PadT): track 0.00 -> 76.8 mm
- net Net-(J1-PadT): track 71.2 -> 0.00 mm
- net Net-(SW1A-C): track 77.1 -> 49.8 mm, vias 0 -> 2
- net Net-(BT1--): track 0.00 -> 18.0 mm
- net 9V: track 192.2 -> 176.7 mm, vias 8 -> 10
- net Net-(BT1-+): track 10.2 -> 13.5 mm
- net /SW_ON: track 63.7 -> 66.4 mm
- net 0: track 23.0 -> 21.5 mm
- net Net-(U1B--): track 21.8 -> 20.6 mm
- net Net-(J3-Pin_1): track 32.7 -> 33.6 mm
- net Net-(J5-Pin_4): track 75.2 -> 76.0 mm
