File: boss_DS1.kicad_sch (KiCad schematic)
At the start: 67 parts, among them J1 NMJ6HHD2, J2 NMJ6HHD2, J3 Conn_01x05, J4 Conn_01x05, J5 Conn_01x05, J6 Barrel_Jack_MountingPin, P1 tube_screamer_front_panel, Q1 MMBT5551, Q2 MMBT5551, Q3 MMBT5551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

Commit message: Init.
Parts:
- removed C1: 47n, Capacitor_SMD:C_0603_1608Metric_Pad1.08x0.95mm_HandSolder, symbol Device:C
- removed C3: 47p, Capacitor_SMD:C_0603_1608Metric_Pad1.08x0.95mm_HandSolder, symbol Device:C
- removed C4, C6: 220n, Capacitor_SMD:C_0603_1608Metric_Pad1.08x0.95mm_HandSolder, symbol Device:C
- removed C5: 100n, Capacitor_SMD:C_0603_1608Metric_Pad1.08x0.95mm_HandSolder, symbol Device:C
- removed D1, D2: 1N4148WS, Diode_SMD:D_SOD-323, symbol Diode:1N4148WS
- removed P1: tube_screamer_front_panel, pedale:tube_screamer_front_plate, symbol pedale:tube_screamer_front_panel
- removed R2: 4.7k, Resistor_SMD:R_0603_1608Metric_Pad0.98x0.95mm_HandSolder, symbol Device:R
- removed R7: 220, Resistor_SMD:R_0603_1608Metric_Pad0.98x0.95mm_HandSolder, symbol Device:R
- added C19, C27: 47n, Capacitor_SMD:C_0603_1608Metric_Pad1.08x0.95mm_HandSolder, symbol Device:C
- added C20: 100p, Capacitor_SMD:C_0603_1608Metric_Pad1.08x0.95mm_HandSolder, symbol Device:C
- added C21: 10n, Capacitor_SMD:C_0603_1608Metric_Pad1.08x0.95mm_HandSolder, symbol Device:C
- added C22: 220p, Capacitor_SMD:C_0603_1608Metric_Pad1.08x0.95mm_HandSolder, symbol Device:C
- added C23, C24: 470n, Capacitor_SMD:C_0603_1608Metric_Pad1.08x0.95mm_HandSolder, symbol Device:C
- added C25: 22n, Capacitor_SMD:C_0603_1608Metric_Pad1.08x0.95mm_HandSolder, symbol Device:C
- added C26: 100n, Capacitor_SMD:C_0603_1608Metric_Pad1.08x0.95mm_HandSolder, symbol Device:C
- added D4, D6, D7: 1N4148WS, Diode_SMD:D_SOD-323, symbol Diode:1N4148WS
- added P1: boss_DS1_front_panel, pedale:boss_DS1_front_plate, symbol pedale:boss_DS1_front_panel
- added Q4: MMBT5551, Package_TO_SOT_SMD:SOT-23, symbol Transistor_BJT:BC817
- added R10, R27: 100k, Resistor_SMD:R_0603_1608Metric_Pad0.98x0.95mm_HandSolder, symbol Device:R
- added R12: 470k, Resistor_SMD:R_0603_1608Metric_Pad0.98x0.95mm_HandSolder, symbol Device:R
- added R24: 22, Resistor_SMD:R_0603_1608Metric_Pad0.98x0.95mm_HandSolder, symbol Device:R
- added R25, R26, R31: 10k, Resistor_SMD:R_0603_1608Metric_Pad0.98x0.95mm_HandSolder, symbol Device:R
- added R28: 2.2k, Resistor_SMD:R_0603_1608Metric_Pad0.98x0.95mm_HandSolder, symbol Device:R
- added R29, R30: 6.8k, Resistor_SMD:R_0603_1608Metric_Pad0.98x0.95mm_HandSolder, symbol Device:R
- added R32, R33, R34: 510k, Resistor_SMD:R_0603_1608Metric_Pad0.98x0.95mm_HandSolder, symbol Device:R
- added R5: 47k, Resistor_SMD:R_0603_1608Metric_Pad0.98x0.95mm_HandSolder, symbol Device:R
- C10: value 1u -> 47n; LCSC C15849 -> C1622
- C11: value 10u -> 1u; LCSC C96446 -> C15849
- C12: value 100n -> 47n; LCSC C14663 -> C1622
- C7: value 1u -> 470n; LCSC C15849 -> C1623
- C9: value 22n -> 47n; LCSC C21122 -> C1622
- R11: value 100 -> 1k; LCSC C22775 -> C21190
- R14: value 1k -> 2.2k; LCSC C21190 -> C4190
- R15: value 510k -> 470k; LCSC C23192 -> C23178
- R21, R3: value 10k -> 100k; LCSC C25804 -> C25803
- R4: value 1k -> 4.7k; LCSC C21190 -> C23162
- R6: value 1k -> 100k; LCSC C21190 -> C25803
- renumbered J4 to J3, J3 to J4
Connections:
- net 0: now also J1.S, J2.S, C21.1, C24.1, D4.2 (A), D6.2 (A), D7.1 (K), R10.2, R24.2; no longer J5.1 (Pin_1)
- net 4V5: now also J5.1 (Pin_1), R15.2, R3.1, C26.2, R27.1, R29.2, R32.1, R33.1; no longer R15.1, R19.1, R3.2, U1.5 (+)
- net 9V: now also R25.1
- net IN_BUFF: now also C23.1, C27.1; no longer C10.1, SW1.3 (C)
- net OP_OUT: now also C21.2, C25.2, D6.1 (K), D7.2 (A), R30.1; no longer J5.3 (Pin_3)
- net SW_MID: now also R34.2
- net SW_ON: now also R31.2; no longer J5.2 (Pin_2)
- net at J4.1 (Pin_1): now also C26.1, R30.2; no longer U1.2 (-)
- net at R4.1: now also C24.2; no longer J3.1 (Pin_1)
- net at C7.1, U1.7: now also J3.1 (Pin_1), C20.1; no longer R6.1
- net at Q2.2 (E), R20.1: now also R11.2; no longer R11.1
- net at C9.2, Q1.1 (B): now also R15.1; no longer R15.2
- net at J3.2 (Pin_2): now also R6.2, C20.2
- net at C11.1: now also R11.1; no longer R11.2
- new net: J4.3 (Pin_3), R28.2, R29.1
- new net: J5.2 (Pin_2), R31.1
- new net: C19.1, C23.2, R27.2
- new net: C19.2, C22.1, Q4.1 (B), R10.1, R12.1
- new net: C22.2, Q4.3 (C), R12.2, R25.2, R26.1
- new net: Q4.2 (E), R24.1
- new net: C10.2, R3.2, R5.1
- new net: R19.1, R32.2
- new net: D4.1 (K), R5.2, U1.3 (+)
- new net: J3.3 (Pin_3), R4.2
- new net: R33.2, R34.1
- new net: C25.1, R28.1
- new net: R6.1, U1.6 (-)
- new net: C27.2, SW1.3 (C)
- new net BJT_GAIN: C10.1, R26.2
- new net OP_BUFF: U1.1, U1.2 (-), U1.5 (+)
- new net TONE_OUT: J4.2 (Pin_2), J5.3 (Pin_3)
Other:
- note added: "BJT and opamp gain stage"
- note added: "Tone control"
- note added: "Volume, output buffer and selection switch"
- note removed: "Clipping and tone stage"
- note removed: "Output buffer and selection switch"
- moved on the sheet: C14, C17, D9, H1, H2, H3, H4, H5, J2, J3, J4, J5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

Commit message: Fix
Parts:
- removed SW1: SW_DPDT_x2, switch:switch_DPDT, symbol Switch:SW_DPDT_x2
- added SW1: pedala_switch, pedale:switch_DPDT, symbol pedale:pedala_switch
Connections:
- net 9V: now also SW1.4 (A)
- net SW_MID: now also SW1.2 (B)
- net SW_ON: now also SW1.1 (A)
- net at C27.2: now also SW1.3 (C)
- net at J5.4 (Pin_4): now also SW1.5 (B)
Changed lines of the file:
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@@
 	)
 	(symbol
+		(lib_id "pedale:pedala_switch")
+		(at 168.91 121.92 0)
+		(mirror y)
+		(unit 1)
+		(exclude_from_sim no)
+		(in_bom yes)
+		(on_board yes)
+		(dnp no)
+		(fields_autoplaced yes)
+		(property "Reference" "SW1"
+			(at 168.91 113.03 0)
+			(effects
+				(font
+					(size 1.27 1.27)
+				)
+			)
+		)
+		(property "Value" "pedala_switch"
+			(at 168.91 115.57 0)
+			(effects
+				(font
+					(size 1.27 1.27)
+				)
+			)
+		)
+		(property "Footprint" "pedale:switch_DPDT"
+			(at 168.91 121.92 0)
+			(effects
+				(font
+					(size 1.27 1.27)
+				)
+				(hide yes)
+			)
+		)
+		(property "Datasheet" "~"
+			(at 168.91 121.92 0)
+			(effects
+				(font
+					(size 1.27 1.27)
+				)
+				(hide yes)
+			)
+		)
+		(property "Description" "Switch, dual pole double throw, separate symbols"
+			(at 168.91 121.92 0)
+			(effects
+				(font
+					(size 1.27 1.27)
+				)
+				(hide yes)
+			)
+		)
+		(pin "6"
+		)
+		(pin "4"
+		)
+		(pin "3"
+		)
+		(pin "5"
+		)
+		(pin "1"
+		)
+		(pin "2"
+		)
+		(instances
+			(project ""
+				(path "/e0801131-6974-42d8-8070-4ed960891aa7"
+					(reference "SW1")
+					(unit 1)
+				)
+			)
+		)
+	)
+	(symbol
 		(lib_id "Simulation_SPICE:0")
 		(at 34.29 168.91 90)
@@
 	)
 	(symbol
-		(lib_id "Switch:SW_DPDT_x2")
-		(at 168.91 121.92 0)
-		(mirror y)
-		(unit 1)
-		(exclude_from_sim no)
-		(in_bom yes)
-		(on_board yes)
-		(dnp no)
-		(property "Reference" "SW1"
-			(at 168.91 113.03 0)
-			(effects
-				(font
-					(size 1.27 1.27)
-				)
-			)
-		)
-		(property "Value" "SW_DPDT_x2"
-			(at 168.91 115.57 0)
-			(effects
-				(font
-					(size 1.27 1.27)
-				)
-			)
-		)
-		(property "Footprint" "switch:switch_DPDT"
-			(at 168.91 121.92 0)
-			(effects
-				(font
-					(size 1.27 1.27)
-				)
-				(hide yes)
-			)
-		)
-		(property "Datasheet" "~"
-			(at 168.91 121.92 0)
-			(effects
-				(font
-					(size 1.27 1.27)
-				)
-				(hide yes)
-			)
-		)
-		(property "Description" "Switch, dual pole double throw, separate symbols"
-			(at 168.91 121.92 0)
-			(effects
-				(font
-					(size 1.27 1.27)
-				)
-				(hide yes)
-			)
-		)
-		(pin "3"
-		)
-		(pin "6"
-		)
-		(pin "5"
-		)
-		(pin "2"
-		)
-		(pin "1"
-		)
-		(pin "4"
-		)
-		(instances
-			(project "tube_screamer"
-				(path "/e0801131-6974-42d8-8070-4ed960891aa7"
-					(reference "SW1")
-					(unit 1)
-				)
-			)
-		)
-	)
-	(symbol
 		(lib_id "Device:R")
 		(at 139.065 41.91 0)
@@
 	)
 	(symbol
-		(lib_id "Switch:SW_DPDT_x2")
-		(at 168.91 106.68 0)
-		(unit 2)
-		(exclude_from_sim no)
-		(in_bom yes)
-		(on_board yes)
-		(dnp no)
-		(property "Reference" "SW1"
-			(at 168.91 97.79 0)
-			(effects
-				(font
-					(size 1.27 1.27)
-				)
-			)
-		)
-		(property "Value" "SW_DPDT_x2"
-			(at 168.91 100.33 0)
-			(effects
-				(font
-					(size 1.27 1.27)
-				)
-			)
-		)
-		(property "Footprint" "switch:switch_DPDT"
-			(at 168.91 106.68 0)
-			(effects
-				(font
-					(size 1.27 1.27)
-				)
-				(hide yes)
-			)
-		)
-		(property "Datasheet" "~"
-			(at 168.91 106.68 0)
-			(effects
-				(font
-					(size 1.27 1.27)
-				)
-				(hide yes)
-			)
-		)
-		(property "Description" "Switch, dual pole double throw, separate symbols"
-			(at 168.91 106.68 0)
-			(effects
-				(font
-					(size 1.27 1.27)
-				)
-				(hide yes)
-			)
-		)
-		(pin "3"
-		)
-		(pin "6"
-		)
-		(pin "5"
-		)
-		(pin "2"
-		)
-		(pin "1"
-		)
-		(pin "4"
-		)
-		(instances
-			(project "tube_screamer"
-				(path "/e0801131-6974-42d8-8070-4ed960891aa7"
-					(reference "SW1")
-					(unit 2)
-				)
-			)
-		)
-	)
-	(symbol
 		(lib_id "Device:Battery_Cell")
 		(at 50.8 181.61 0)
@@
 				)
 			)
+		)
+	)
+	(symbol
+		(lib_id "pedale:pedala_switch")
+		(at 168.91 106.68 0)
+		(unit 2)
+		(exclude_from_sim no)
+		(in_bom yes)
+		(on_board yes)
+		(dnp no)
+		(fields_autoplaced yes)
+		(property "Reference" "SW1"
+			(at 168.91 97.79 0)
+			(effects
+				(font
+					(size 1.27 1.27)
+				)
+			)
+		)
+		(property "Value" "pedala_switch"
+			(at 168.91 100.33 0)
+			(effects
+				(font
+					(size 1.27 1.27)
+				)
+			)
+		)
+		(property "Footprint" "pedale:switch_DPDT"
+			(at 168.91 106.68 0)
+			(effects
+				(font
+					(size 1.27 1.27)
+				)
+				(hide yes)
+			)
+		)
+		(property "Datasheet" "~"
+			(at 168.91 106.68 0)
+			(effects
+				(font
+					(size 1.27 1.27)
+				)
+				(hide yes)
+			)
+		)
+		(property "Description" "Switch, dual pole double throw, separate symbols"
+			(at 168.91 106.68 0)
+			(effects
+				(font
+					(size 1.27 1.27)
+				)
+				(hide yes)
+			)
+		)
+		(pin "6"
+		)
+		(pin "4"
+		)
+		(pin "3"
+		)
+		(pin "5"
+		)
+		(pin "1"
+		)
+		(pin "2"
+		)
+		(instances
+			(project ""
+				(path "/e0801131-6974-42d8-8070-4ed960891aa7"
+					(reference "SW1")
+					(unit 2)
+				)
+			)

Commit message: oK
Parts:
- removed R26: 10k, Resistor_SMD:R_0603_1608Metric_Pad0.98x0.95mm_HandSolder, symbol Device:R
Connections:
- net 0: no longer D6.2 (A), D7.1 (K)
- net 4V5: now also D6.2 (A), D7.1 (K)
- net BJT_GAIN: now also C22.2, Q4.3 (C), R12.2, R25.2
Changed lines of the file:
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@@
 		(color 0 0 0 0)
 	)
+	(junction
+		(at 254 78.74)
+		(diameter 0)
+		(color 0 0 0 0)
+	)
 	(no_connect
 		(at 173.99 109.22)
@@
 	(wire
 		(pts
-			(xy 260.35 76.2) (xy 260.35 77.47)
-		)
-		(stroke
-			(width 0)
-			(type default)
-		)
-	)
-	(wire
-		(pts
 			(xy 196.85 109.22) (xy 196.85 105.41)
 		)
@@
 	(wire
 		(pts
-			(xy 254 76.2) (xy 254 77.47)
-		)
-		(stroke
-			(width 0)
-			(type default)
-		)
-	)
-	(wire
-		(pts
 			(xy 76.2 118.11) (xy 50.8 118.11)
 		)
@@
 	(wire
 		(pts
-			(xy 182.245 48.26) (xy 184.785 48.26)
+			(xy 233.68 52.07) (xy 226.06 52.07)
 		)
 		(stroke
@@
 	(wire
 		(pts
-			(xy 233.68 52.07) (xy 226.06 52.07)
+			(xy 260.35 76.2) (xy 260.35 78.74)
 		)
 		(stroke
@@
 	(wire
 		(pts
+			(xy 254 76.2) (xy 254 78.74)
+		)
+		(stroke
+			(width 0)
+			(type default)
+		)
+	)
+	(wire
+		(pts
 			(xy 111.76 184.15) (xy 111.76 189.23)
 		)
@@
 	(wire
 		(pts
-			(xy 170.18 48.26) (xy 174.625 48.26)
+			(xy 170.18 48.26) (xy 176.53 48.26)
 		)
 		(stroke
@@
 	(wire
 		(pts
+			(xy 247.65 78.74) (xy 254 78.74)
+		)
+		(stroke
+			(width 0)
+			(type default)
+		)
+	)
+	(wire
+		(pts
 			(xy 72.39 125.73) (xy 76.2 125.73)
 		)
@@
 	(wire
 		(pts
+			(xy 254 78.74) (xy 260.35 78.74)
+		)
+		(stroke
+			(width 0)
+			(type default)
+		)
+	)
+	(wire
+		(pts
 			(xy 260.35 64.77) (xy 266.7 64.77)
 		)
@@
 	(global_label "4V5"
 		(shape input)
+		(at 247.65 78.74 180)
+		(fields_autoplaced yes)
+		(effects
+			(font
+				(size 1.27 1.27)
+			)
+			(justify right)
+		)
+		(property "Intersheetrefs" "${INTERSHEET_REFS}"
+			(at 241.1572 78.74 0)
+			(effects
+				(font
+					(size 1.27 1.27)
+				)
+				(justify right)
+				(hide yes)
+			)
+		)
+	)
+	(global_label "4V5"
+		(shape input)
 		(at 140.335 31.75 0)
 		(fields_autoplaced yes)
@@
 	(global_label "BJT_GAIN"
 		(shape output)
-		(at 184.785 48.26 0)
+		(at 176.53 48.26 0)
 		(fields_autoplaced yes)
 		(effects
@@
 		)
 		(property "Intersheetrefs" "${INTERSHEET_REFS}"
-			(at 196.2369 48.26 0)
+			(at 187.9819 48.26 0)
 			(effects
 				(font
@@
 	)
 	(symbol
-		(lib_id "Simulation_SPICE:0")
-		(at 260.35 77.47 0)
-		(mirror y)
-		(unit 1)
-		(exclude_from_sim no)
-		(in_bom yes)
-		(on_board yes)
-		(dnp no)
-		(property "Reference" "#GND030"
-			(at 260.35 80.01 0)
-			(effects
-				(font
-					(size 1.27 1.27)
-				)
-				(hide yes)
-			)
-		)
-		(property "Value" "0"
-			(at 278.13 78.74 0)
-			(effects
-				(font
-					(size 1.27 1.27)
-				)
-				(hide yes)
-			)
-		)
-		(property "Footprint" ""
-			(at 260.35 77.47 0)
-			(effects
-				(font
-					(size 1.27 1.27)
-				)
-				(hide yes)
-			)
-		)
-		(property "Datasheet" "~"
-			(at 260.35 77.47 0)
-			(effects
-				(font
-					(size 1.27 1.27)
-				)
-				(hide yes)
-			)
-		)
-		(property "Description" ""
-			(at 260.35 77.47 0)
-			(effects
-				(font
-					(size 1.27 1.27)
-				)
-			)
-		)
-		(pin "1"
-		)
-		(instances
-			(project "boss_DS1"
-				(path "/e0801131-6974-42d8-8070-4ed960891aa7"
-					(reference "#GND030")
-					(unit 1)
-				)
-			)
-		)
-	)
-	(symbol
 		(lib_id "Graphic:Logo_Open_Hardware_Small")
 		(at 273.05 157.48 0)
@@
 	)
 	(symbol
-		(lib_id "Simulation_SPICE:0")
-		(at 254 77.47 0)
-		(unit 1)
-		(exclude_from_sim no)
-		(in_bom yes)
-		(on_board yes)
-		(dnp no)
-		(property "Reference" "#GND029"
-			(at 254 80.01 0)
-			(effects
-				(font
-					(size 1.27 1.27)
-				)
-				(hide yes)
-			)
-		)
-		(property "Value" "0"
-			(at 236.22 78.74 0)
-			(effects
-				(font
-					(size 1.27 1.27)
-				)
-				(hide yes)
-			)
-		)
-		(property "Footprint" ""
-			(at 254 77.47 0)
-			(effects
-				(font
-					(size 1.27 1.27)
-				)
-				(hide yes)
-			)
-		)
-		(property "Datasheet" "~"
-			(at 254 77.47 0)
-			(effects
-				(font
-					(size 1.27 1.27)
-				)
-				(hide yes)
-			)
-		)
-		(property "Description" ""
-			(at 254 77.47 0)
-			(effects
-				(font
-					(size 1.27 1.27)
-				)
-			)
-		)
-		(pin "1"
-		)
-		(instances
-			(project "boss_DS1"
-				(path "/e0801131-6974-42d8-8070-4ed960891aa7"
-					(reference "#GND029")
-					(unit 1)
-				)
-			)
-		)
-	)
-	(symbol
 		(lib_id "Device:R")
 		(at 69.85 128.27 270)
@@
 					(unit 1)
 				)
-			)
-		)
-	)
-	(symbol
-		(lib_id "Device:R")
-		(at 178.435 48.26 90)
-		(unit 1)
-		(exclude_from_sim no)
-		(in_bom yes)
-		(on_board yes)
-		(dnp no)
-		(fields_autoplaced yes)
-		(property "Reference" "R26"
-			(at 178.435 41.91 90)
-			(effects
-				(font
-					(size 1.27 1.27)
-				)
-			)
-		)
-		(property "Value" "10k"
-			(at 178.435 44.45 90)
-			(effects
-				(font
-					(size 1.27 1.27)
-				)
-			)
-		)
-		(property "Footprint" "Resistor_SMD:R_0603_1608Metric_Pad0.98x0.95mm_HandSolder"
-			(at 178.435 50.038 90)
-			(effects
-				(font
-					(size 1.27 1.27)
-				)
-				(hide yes)
-			)
-		)
-		(property "Datasheet" "~"
-			(at 178.435 48.26 0)
-			(effects
-				(font
-					(size 1.27 1.27)
-				)
-				(hide yes)
-			)
-		)
-		(property "Description" ""
-			(at 178.435 48.26 0)
-			(effects
-				(font
-					(size 1.27 1.27)
-				)
-			)
-		)
-		(property "LCSC" "C25804"
-			(at 178.435 48.26 0)
-			(effects
-				(font
-					(size 1.27 1.27)
-				)
-				(hide yes)
-			)
-		)
-		(pin "1"
-		)
-		(pin "2"
-		)
-		(instances
-			(project "boss_DS1"
-				(path "/e0801131-6974-42d8-8070-4ed960891aa7"
-					(reference "R26")
-					(unit 1)
-				)

Commit message: All errors fixed
Parts:
- removed J1, J2: NMJ6HHD2, Connector_Audio:Jack_6.35mm_Neutrik_NMJ6HHD2_Horizontal, symbol Connector_Audio:NMJ6HHD2
- removed J6: Barrel_Jack_MountingPin, Connector_BarrelJack:BarrelJack_GCT_DCJ200-10-A_Horizontal, symbol Connector:Barrel_Jack_MountingPin
- removed RV7, RV9: floating_pot_knob, pedale:floating_pot_knob, symbol pedale:floating_pot_knob
- added J2, J6: Jack_6.35, pedale:Jack_6.35mm, symbol pedale:Jack_6.35
- added J7, J8: Conn_01x01_Socket, TestPoint:TestPoint_THTPad_D2.5mm_Drill1.2mm, symbol Connector:Conn_01x01_Socket
- added J9: Barrel_Jack_Switch, pedale:BarrelJack, symbol Connector:Barrel_Jack_Switch
- SW1: footprint pedale:switch_DPDT -> pedale:foot_switch_tht_and_floating
Connections:
- net 0: now also J2.R, J2.S, J6.R, J6.S, J9.2; no longer BT1.2 (-)
- net at BT1.1 (+), D5.2 (A): now also J7.1 (Pin_1)
- net at C11.2, R21.1: now also J2.T
- net at R13.2: now also J6.T
- net at D3.2 (A): now also J9.1
- new net: BT1.2 (-), J8.1 (Pin_1), J9.3
- no-connect marks 4 -> 3
Other:
- moved on the sheet: D8
